File: xt60_adapter/xt60_adapter/xt60_adapter.kicad_sch (KiCad schematic)
At the start: 3 parts, among them J1 Barrel_Jack_Switch, J2 Conn_01x02

Commit message: Add projects
Connections:
- net GND: now reaches C1.2, J1.2, J2.1 (Pin_1)
Changed lines of the file:
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@@
+    (stroke (width 0) (type default) (color 0 0 0 0))
+  )
+  (wire (pts (xy 96.52 63.5) (xy 104.14 63.5))
     (stroke (width 0) (type default) (color 0 0 0 0))
   )
@@
   )
   (wire (pts (xy 82.55 69.85) (xy 104.14 69.85))
+    (stroke (width 0) (type default) (color 0 0 0 0))
+  )
+  (wire (pts (xy 104.14 63.5) (xy 104.14 69.85))
     (stroke (width 0) (type default) (color 0 0 0 0))
   )
@@
     (pin "3")
   )
+  (symbol (lib_id "power:GND") (at 96.52 63.5 0) (unit 1)
+    (in_bom yes) (on_board yes) (fields_autoplaced)
+    (property "Reference" "#PWR?" (id 0) (at 96.52 69.85 0)
+      (effects (font (size 1.27 1.27)) hide)
+    )
+    (property "Value" "GND" (id 1) (at 96.52 68.58 0))
+    (property "Footprint" "" (id 2) (at 96.52 63.5 0)
+      (effects (font (size 1.27 1.27)) hide)
+    )
+    (property "Datasheet" "" (id 3) (at 96.52 63.5 0)
+      (effects (font (size 1.27 1.27)) hide)
+    )
+    (pin "1")
+  )
   (sheet_instances
     (path "/" (page "1"))
   )
   (symbol_instances
+    (path "/82094c54-4e68-497e-b2df-a34cc5f32d0f"
+      (reference "#PWR?") (unit 1) (value "GND") (footprint "")
+    )
     (path "/3baf2eac-0bea-426c-94bc-f645721424c0"
       (reference "C1") (unit 1) (value "1000u") (footprint "Capacitor_THT:CP_Radial_D16.0mm_P7.50mm")
