File: doom_day_lamp/doom_day_lamp/doom_day_lamp.kicad_pcb (KiCad board)
At the start: 2 copper layers, 21 parts, among them J1 Conn_01x02_Female

Commit message: Add projects
Parts:
- added D11: LED, LED_THT:LED_D3.0mm, F.Cu at (58.4, 52.1)
- added D12: LED, LED_THT:LED_D3.0mm, F.Cu at (67.3, 52.1)
- added D13: LED, LED_THT:LED_D3.0mm, F.Cu at (76.2, 52.1)
- added D14: LED, LED_THT:LED_D3.0mm, F.Cu at (85.1, 52.1)
- added D15: LED, LED_THT:LED_D3.0mm, F.Cu at (94.0, 52.1)
- added D16: LED, LED_THT:LED_D3.0mm, F.Cu at (102.9, 52.1)
- added D17: LED, LED_THT:LED_D3.0mm, F.Cu at (111.8, 52.1)
- added D18: LED, LED_THT:LED_D3.0mm, F.Cu at (120.7, 52.1)
- added D19: LED, LED_THT:LED_D3.0mm, F.Cu at (129.5, 52.1)
- added D20: LED, LED_THT:LED_D3.0mm, F.Cu at (138.4, 52.1)
- added JP1: Jumper_2_Bridged, Connector_PinHeader_2.54mm:PinHeader_1x02_P2.54mm_Vertical, F.Cu at (152.4, 59.7)
- added R11: 16, Resistor_THT:R_Axial_DIN0207_L6.3mm_D2.5mm_P2.54mm_Vertical, F.Cu at (62.9, 49.5)
- added R12: 16, Resistor_THT:R_Axial_DIN0207_L6.3mm_D2.5mm_P2.54mm_Vertical, F.Cu at (71.8, 49.5)
- added R13: 16, Resistor_THT:R_Axial_DIN0207_L6.3mm_D2.5mm_P2.54mm_Vertical, F.Cu at (80.6, 49.5)
- added R14: 16, Resistor_THT:R_Axial_DIN0207_L6.3mm_D2.5mm_P2.54mm_Vertical, F.Cu at (89.5, 49.5)
- added R15: 16, Resistor_THT:R_Axial_DIN0207_L6.3mm_D2.5mm_P2.54mm_Vertical, F.Cu at (98.4, 49.5)
- added R16: 16, Resistor_THT:R_Axial_DIN0207_L6.3mm_D2.5mm_P2.54mm_Vertical, F.Cu at (107.3, 49.5)
- added R17: 16, Resistor_THT:R_Axial_DIN0207_L6.3mm_D2.5mm_P2.54mm_Vertical, F.Cu at (116.2, 49.5)
- added R18: 16, Resistor_THT:R_Axial_DIN0207_L6.3mm_D2.5mm_P2.54mm_Vertical, F.Cu at (125.1, 49.5)
- added R19: 16, Resistor_THT:R_Axial_DIN0207_L6.3mm_D2.5mm_P2.54mm_Vertical, F.Cu at (134.0, 49.5)
- added R20: 16, Resistor_THT:R_Axial_DIN0207_L6.3mm_D2.5mm_P2.54mm_Vertical, F.Cu at (142.9, 49.5)
- added SW1: SW_Push_SPDT, _switch:SW_CuK_OS102011MA1QN1_SPDT_Angled, F.Cu at (156.8, 59.8)
- added U1: Mini360, _dc_dc_converters:Mini360_step-down, F.Cu at (157.5, 50.2)
- J1: footprint Connector_AMASS:AMASS_XT30U-M_1x02_P5.0mm_Vertical -> Connector_PinHeader_2.00mm:PinHeader_1x02_P2.00mm_Vertical
- R1, R10, R2, R3, R4, R5, R6, R7, R8, R9: footprint Resistor_THT:R_Axial_DIN0207_L6.3mm_D2.5mm_P7.62mm_Horizontal -> Resistor_THT:R_Axial_DIN0207_L6.3mm_D2.5mm_P2.54mm_Vertical
- moved J1 156.3 mm to (174.6, 52.3), turned to 0 degrees
- moved R10 115.0 mm to (145.4, 57.1), turned to -90 degrees
- moved R1 109.7 mm to (136.5, 57.1), turned to -90 degrees
- moved D1 103.6 mm to (141.0, 54.6), turned to -90 degrees
- moved D2 99.2 mm to (132.1, 54.6), turned to -90 degrees
- moved R3 89.8 mm to (118.7, 57.1), turned to -90 degrees
- moved D3 83.5 mm to (123.2, 54.6), turned to -90 degrees
- moved D4 78.9 mm to (114.3, 54.6), turned to -90 degrees
- moved R2 73.2 mm to (127.6, 57.1), turned to -90 degrees
- moved D5 62.9 mm to (105.4, 54.6), turned to -90 degrees
- moved R8 56.7 mm to (74.3, 57.1), turned to -90 degrees
- moved R4 52.7 mm to (109.9, 57.1), turned to -90 degrees
- moved D6 52.7 mm to (96.5, 54.6), turned to -90 degrees
- moved D7 49.0 mm to (87.6, 54.6), turned to -90 degrees
- moved D8 44.1 mm to (78.7, 54.6), turned to -90 degrees
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Connections:
- D1 pad 1: GND -> GND1
- D10 pad 1: GND -> GND1
- D2 pad 1: GND -> GND1
- D3 pad 1: GND -> GND1
- D4 pad 1: GND -> GND1
- D5 pad 1: GND -> GND1
- D6 pad 1: GND -> GND1
- D7 pad 1: GND -> GND1
- D8 pad 1: GND -> GND1
- D9 pad 1: GND -> GND1
- J1 pad 2: +12V -> Net-(J1-Pad2)
- R1 pad 2: +12V -> Net-(JP1-Pad2)
- R10 pad 2: +12V -> Net-(JP1-Pad2)
- R2 pad 2: +12V -> Net-(JP1-Pad2)
- R3 pad 2: +12V -> Net-(JP1-Pad2)
- R4 pad 2: +12V -> Net-(JP1-Pad2)
- R5 pad 2: +12V -> Net-(JP1-Pad2)
- R6 pad 2: +12V -> Net-(JP1-Pad2)
- R7 pad 2: +12V -> Net-(JP1-Pad2)
- R8 pad 2: +12V -> Net-(JP1-Pad2)
- R9 pad 2: +12V -> Net-(JP1-Pad2)
Routing:
- net Net-(JP1-Pad2): track 0.00 -> 188.3 mm
- net Net-(JP1-Pad1): track 0.00 -> 18.2 mm
- net Net-(SW1-Pad1): track 0.00 -> 16.3 mm
- net Net-(J1-Pad2): track 0.00 -> 13.8 mm
- net Net-(D19-Pad2): track 0.00 -> 4.45 mm
- net Net-(D9-Pad2): track 0.00 -> 4.45 mm
- net Net-(D8-Pad2): track 0.00 -> 4.45 mm
- net Net-(D7-Pad2): track 0.00 -> 4.45 mm
- net Net-(D6-Pad2): track 0.00 -> 4.45 mm
- net Net-(D5-Pad2): track 0.00 -> 4.45 mm
- net Net-(D4-Pad2): track 0.00 -> 4.45 mm
- net Net-(D3-Pad2): track 0.00 -> 4.45 mm
- net Net-(D11-Pad2): track 0.00 -> 4.45 mm
- net Net-(D10-Pad2): track 0.00 -> 4.45 mm
- net Net-(D20-Pad2): track 0.00 -> 4.44 mm
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- added copper zone on B.Cu, net (none)
- added copper zone on B.Cu, net GND
- added copper zone on B.Cu, net GND1
Other:
- board outline added: 130.1 x 18 mm

Commit message: Update lamp
Parts:
- moved J1 3.86 mm to (170.8, 51.7)
Connections:
- D1 pad 1: GND1 -> GND
- D10 pad 1: GND1 -> GND
- D11 pad 1: GND1 -> GND
- D12 pad 1: GND1 -> GND
- D13 pad 1: GND1 -> GND
- D14 pad 1: GND1 -> GND
- D15 pad 1: GND1 -> GND
- D16 pad 1: GND1 -> GND
- D17 pad 1: GND1 -> GND
- D18 pad 1: GND1 -> GND
- D19 pad 1: GND1 -> GND
- D2 pad 1: GND1 -> GND
- D20 pad 1: GND1 -> GND
- D3 pad 1: GND1 -> GND
- D4 pad 1: GND1 -> GND
- D5 pad 1: GND1 -> GND
- D6 pad 1: GND1 -> GND
- D7 pad 1: GND1 -> GND
- D8 pad 1: GND1 -> GND
- D9 pad 1: GND1 -> GND
- U1 pad 3: GND1 -> GND
Routing:
- net Net-(J1-Pad2): track 13.8 -> 11.5 mm
- net (no net): vias 4 -> 0
- removed copper zone on B.Cu, net (none)
- removed copper zone on B.Cu, net GND1
Other:
- board size 130.1 x 18 mm -> 124.5 x 19.1 mm
