File: amp/amp/amp.kicad_sch (KiCad schematic)
At the start: 7 parts, among them J1 Conn_01x02_Female, J2 TSJ3.5-009, J3 Screw_Terminal_01x02, J4 Screw_Terminal_01x02

Commit message: Add projects
Parts:
- removed DC1: mp1584, _DC_DC:MP1584, symbol _dc_dc:mp1584
- removed J1: Conn_01x02_Female, Connector_PinSocket_2.00mm:PinSocket_1x02_P2.00mm_Vertical, symbol Connector:Conn_01x02_Female
- added J1: Conn_01x02, Connector_JST:JST_PH_B2B-PH-K_1x02_P2.00mm_Vertical, symbol Connector_Generic:Conn_01x02
Connections:
- net GND: now also J1.1 (Pin_1)
- net at AMP1.4 (5v+), C1.1: now also J1.2 (Pin_2)
Other:
- moved on the sheet: C1
