File: dc_ph2_converter/dc_ph2_converter/dc_ph2_converter.kicad_pcb (KiCad board)
At the start: 2 copper layers, 33.7 x 21.6 mm, 3 parts, among them J1 Barrel_Jack_MountingPin, J2 Conn_01x02

Commit message: Add projects
Parts:
- removed C1: C_Polarized, Capacitor_THT:CP_Radial_D12.5mm_P5.00mm
- added J3: Conn_01x02, Connector_JST:JST_PH_B2B-PH-K_1x02_P2.00mm_Vertical, F.Cu at (112.3, 71.7)
- added J4: Conn_01x02, Connector_JST:JST_PH_B2B-PH-K_1x02_P2.00mm_Vertical, F.Cu at (105.3, 71.7)
- added J5: Conn_01x02, Connector_JST:JST_PH_B2B-PH-K_1x02_P2.00mm_Vertical, F.Cu at (105.4, 63.5)
- J2: footprint Connector_PinHeader_2.00mm:PinHeader_1x02_P2.00mm_Vertical -> Connector_JST:JST_PH_B2B-PH-K_1x02_P2.00mm_Vertical
- moved J2 9.21 mm to (112.4, 63.5), turned to -90 degrees
Connections:
- J1 pad 1: Net-(C1-Pad1) -> Net-(J1-Pad1)
- J2 pad 1: Net-(C1-Pad1) -> GND
- J2 pad 2: GND -> Net-(J1-Pad1)
Routing:
- net Net-(J1-Pad1): track 0.00 -> 33.6 mm
- net Net-(C1-Pad1): track 23.0 -> 0.00 mm
- added copper zone on B.Cu, net GND
- removed copper zone on F.Cu, net GND
Other:
- board size 33.7 x 21.6 mm -> 31.8 x 22.9 mm

Commit message: Add dc_ph2
Parts:
- added ?: , , F.Cu at (116.8, 78.7)
- added ?: , , F.Cu at (93.3, 78.7)
- added ?: , , F.Cu at (116.8, 58.4)
- added REF**: MountingHole_3.2mm_M3_ISO14580_Pad, MountingHole:MountingHole_3.2mm_M3_ISO14580_Pad, F.Cu at (93.3, 58.4)
Other:
- board size 31.8 x 22.9 mm -> 32.4 x 29.2 mm
Changed lines of the file:
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@@
   (net 1 "GND")
   (net 2 "Net-(J1-Pad1)")
+  (footprint "MountingHole:MountingHole_3.2mm_M3_ISO14580_Pad" (layer "F.Cu")
+    (at 93.345 58.42)
+    (descr "Mounting Hole 3.2mm, M3, ISO14580")
+    (tags "mounting hole 3.2mm m3 iso14580")
+    (attr exclude_from_pos_files exclude_from_bom)
+    (fp_text reference "REF**" (at 0 -3.75) (layer "F.SilkS")
+      (effects (font (size 1 1) (thickness 0.15)))
+    )
+    (fp_text value "MountingHole_3.2mm_M3_ISO14580_Pad" (at 0 3.75) (layer "F.Fab")
+      (effects (font (size 1 1) (thickness 0.15)))
+    )
+    (fp_text user "${REFERENCE}" (at 0 0) (layer "F.Fab")
+      (effects (font (size 1 1) (thickness 0.15)))
+    )
+    (fp_circle (center 0 0) (end 2.75 0) (layer "Cmts.User") (width 0.15) (fill none))
+    (fp_circle (center 0 0) (end 3 0) (layer "F.CrtYd") (width 0.05) (fill none))
+    (pad "1" thru_hole circle (at 0 0) (size 5.5 5.5) (drill 3.2) (layers *.Cu *.Mask))
+  )
+  (footprint "" (layer "F.Cu")
+    (at 116.84 78.74)
+    (fp_text reference "" (at 0 0) (layer "F.SilkS")
+      (effects (font (size 1.27 1.27) (thickness 0.15)))
+    )
+    (fp_text value "" (at 0 0) (layer "F.SilkS")
+      (effects (font (size 1.27 1.27) (thickness 0.15)))
+    )
+    (pad "1" thru_hole circle (at 0 0) (size 5.5 5.5) (drill 3.2) (layers *.Cu *.Mask))
+  )
+  (footprint "" (layer "F.Cu")
+    (at 93.345 78.74)
+    (fp_text reference "" (at 0 0) (layer "F.SilkS")
+      (effects (font (size 1.27 1.27) (thickness 0.15)))
+    )
+    (fp_text value "" (at 0 0) (layer "F.SilkS")
+      (effects (font (size 1.27 1.27) (thickness 0.15)))
+    )
+    (pad "1" thru_hole circle (at 0 0) (size 5.5 5.5) (drill 3.2) (layers *.Cu *.Mask))
+  )
   (footprint "Connector_JST:JST_PH_B2B-PH-K_1x02_P2.00mm_Vertical" (layer "F.Cu")
     (at 112.395 63.5 -90)
@@
     (fp_line (start -2.36 -2.11) (end -2.36 -0.86) (layer "F.Fab") (width 0.1))
     (fp_line (start -1.95 -1.7) (end -1.95 2.8) (layer "F.Fab") (width 0.1))
-    (pad "1" thru_hole roundrect (at 0 0 270) (size 1.5 1.75) (drill 0.8) (layers *.Cu *.Mask) (roundrect_rratio 0.208333)
+    (pad "1" thru_hole roundrect (at 0 0 270) (size 1.5 1.75) (drill 0.8) (layers *.Cu *.Mask) (roundrect_rratio 0.2083333333)
       (net 1 "GND") (pinfunction "Pin_1") (pintype "passive"))
     (pad "2" thru_hole oval (at 2 0 270) (size 1.5 1.75) (drill 0.8) (layers *.Cu *.Mask)
@@
       (rotate (xyz 0 0 0))
     )
+  )
+  (footprint "" (layer "F.Cu")
+    (at 116.84 58.42)
+    (fp_text reference "" (at 0 0) (layer "F.SilkS")
+      (effects (font (size 1.27 1.27) (thickness 0.15)))
+    )
+    (fp_text value "" (at 0 0) (layer "F.SilkS")
+      (effects (font (size 1.27 1.27) (thickness 0.15)))
+    )
+    (pad "1" thru_hole circle (at 0 0) (size 5.5 5.5) (drill 3.2) (layers *.Cu *.Mask))
   )
   (footprint "Connector_JST:JST_PH_B2B-PH-K_1x02_P2.00mm_Vertical" (layer "F.Cu")
@@
     (fp_line (start 3.95 2.8) (end 3.95 -1.7) (layer "F.Fab") (width 0.1))
     (fp_line (start -1.11 -2.11) (end -2.36 -2.11) (layer "F.Fab") (width 0.1))
-    (pad "1" thru_hole roundrect (at 0 0 270) (size 1.5 1.75) (drill 0.8) (layers *.Cu *.Mask) (roundrect_rratio 0.208333)
+    (pad "1" thru_hole roundrect (at 0 0 270) (size 1.5 1.75) (drill 0.8) (layers *.Cu *.Mask) (roundrect_rratio 0.2083333333)
       (net 1 "GND") (pinfunction "Pin_1") (pintype "passive"))
     (pad "2" thru_hole oval (at 2 0 270) (size 1.5 1.75) (drill 0.8) (layers *.Cu *.Mask)
@@
     (fp_line (start 3.95 -1.7) (end -1.95 -1.7) (layer "F.Fab") (width 0.1))
     (fp_line (start -1.95 -1.7) (end -1.95 2.8) (layer "F.Fab") (width 0.1))
-    (pad "1" thru_hole roundrect (at 0 0 270) (size 1.5 1.75) (drill 0.8) (layers *.Cu *.Mask) (roundrect_rratio 0.208333)
+    (pad "1" thru_hole roundrect (at 0 0 270) (size 1.5 1.75) (drill 0.8) (layers *.Cu *.Mask) (roundrect_rratio 0.2083333333)
       (net 1 "GND") (pinfunction "Pin_1") (pintype "passive"))
     (pad "2" thru_hole oval (at 2 0 270) (size 1.5 1.75) (drill 0.8) (layers *.Cu *.Mask)
@@
     (fp_line (start -1.11 -2.11) (end -2.36 -2.11) (layer "F.Fab") (width 0.1))
     (fp_line (start -1.95 2.8) (end 3.95 2.8) (layer "F.Fab") (width 0.1))
-    (pad "1" thru_hole roundrect (at 0 0 270) (size 1.5 1.75) (drill 0.8) (layers *.Cu *.Mask) (roundrect_rratio 0.208333)
+    (pad "1" thru_hole roundrect (at 0 0 270) (size 1.5 1.75) (drill 0.8) (layers *.Cu *.Mask) (roundrect_rratio 0.2083333333)
       (net 1 "GND") (pinfunction "Pin_1") (pintype "passive"))
     (pad "2" thru_hole oval (at 2 0 270) (size 1.5 1.75) (drill 0.8) (layers *.Cu *.Mask)
@@
     )
   )
-  (gr_circle (center 117.475 60.325) (end 118.275 60.325) (layer "Edge.Cuts") (width 0.1) (fill none))
-  (gr_circle (center 117.475 60.325) (end 118.975 60.325) (layer "Edge.Cuts") (width 0.1) (fill none))
-  (gr_circle (center 117.475 76.835) (end 118.975 76.835) (layer "Edge.Cuts") (width 0.1) (fill none))
-  (gr_circle (center 92.075 76.835) (end 93.575 76.835) (layer "Edge.Cuts") (width 0.1) (fill none))
-  (gr_circle (center 92.075 60.325) (end 93.575 60.325) (layer "Edge.Cuts") (width 0.1) (fill none))
-  (gr_line (start 120.65 76.835) (end 120.65 60.325) (layer "Edge.Cuts") (width 0.1))
-  (gr_circle (center 117.475 76.835) (end 118.275 76.835) (layer "Edge.Cuts") (width 0.1) (fill none))
-  (gr_arc (start 117.475 57.15) (mid 119.720064 58.079936) (end 120.65 60.325) (layer "Edge.Cuts") (width 0.1))
-  (gr_arc (start 92.075 80.01) (mid 89.829936 79.080064) (end 88.9 76.835) (layer "Edge.Cuts") (width 0.1))
-  (gr_line (start 117.475 80.01) (end 92.075 80.01) (layer "Edge.Cuts") (width 0.1))
-  (gr_line (start 117.475 57.15) (end 92.075 57.15) (layer "Edge.Cuts") (width 0.1))
-  (gr_arc (start 120.65 76.835) (mid 119.720064 79.080064) (end 117.475 80.01) (layer "Edge.Cuts") (width 0.1))
-  (gr_arc (start 88.9 60.325) (mid 89.829936 58.079936) (end 92.075 57.15) (layer "Edge.Cuts") (width 0.1))
-  (gr_circle (center 92.075 76.835) (end 92.875 76.835) (layer "Edge.Cuts") (width 0.1) (fill none))
-  (gr_circle (center 92.075 60.325) (end 92.875 60.325) (layer "Edge.Cuts") (width 0.1) (fill none))
-  (gr_line (start 88.9 60.325) (end 88.9 76.835) (layer "Edge.Cuts") (width 0.1))
+  (gr_arc (start 116.84 53.975) (mid 119.98309 55.27691) (end 121.285 58.42) (layer "Edge.Cuts") (width 0.1))
+  (gr_arc (start 88.9 58.42) (mid 90.20191 55.27691) (end 93.345 53.975) (layer "Edge.Cuts") (width 0.1))
+  (gr_arc (start 121.285 78.74) (mid 119.98309 81.88309) (end 116.84 83.185) (layer "Edge.Cuts") (width 0.1))
+  (gr_line (start 121.285 78.74) (end 121.285 58.42) (layer "Edge.Cuts") (width 0.1))
+  (gr_line (start 116.84 83.185) (end 93.345 83.185) (layer "Edge.Cuts") (width 0.1))
+  (gr_line (start 116.84 53.975) (end 93.345 53.975) (layer "Edge.Cuts") (width 0.1))
+  (gr_arc (start 93.345 83.185) (mid 90.20191 81.88309) (end 88.9 78.74) (layer "Edge.Cuts") (width 0.1))
+  (gr_line (start 88.9 58.42) (end 88.9 78.74) (layer "Edge.Cuts") (width 0.1))
   (segment (start 99.06 67.93) (end 99.06 69.215) (width 0.25) (layer "F.Cu") (net 2))
   (segment (start 99.06 67.93) (end 99.06 66.675) (width 0.25) (layer "F.Cu") (net 2))
@@
   (segment (start 99.06 67.93) (end 99.06 69.85) (width 0.25) (layer "B.Cu") (net 2))
   (zone (net 1) (net_name "GND") (layer "B.Cu") (hatch edge 0.508)
-    (connect_pads (clearance 0.508))
+    (connect_pads (clearance 1.1))
     (min_thickness 0.254) (filled_areas_thickness no)
-    (fill yes (thermal_gap 0.508) (thermal_bridge_width 0.508))
+    (fill yes (thermal_gap 0.75) (thermal_bridge_width 0.508))
     (polygon
       (pts
-        (xy 121.92 80.01)
-        (xy 88.9 80.01)
-        (xy 88.9 57.15)
-        (xy 121.92 57.15)
+        (xy 121.285 83.82)
+        (xy 88.265 83.82)
+        (xy 88.265 53.34)
+        (xy 121.285 53.34)
       )
     )
